File: SmartPortAdapter.kicad_sch (KiCad schematic)
At the start: 9 parts, among them J1 APPLE_SDISKII, J2 Data Pin, J3 PHx/SEL

Commit message: initial commit
Other:
- title: (none) -> SmartPortAdapter
Changed lines of the file:
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@@
 	(generator_version "8.0")
 	(paper "A4")
+	(title_block
+		(title "SmartPortAdapter")
+		(rev "1")
+	)
 	(junction
 		(at 104.14 59.69)

Commit message: rev3 IIGS ROM3
Parts:
- removed J2: Data Pin, Connector_PinHeader_2.54mm:PinHeader_1x06_P2.54mm_Vertical, symbol Connector_Generic:Conn_01x06
- removed J3: PHx/SEL, Connector_PinHeader_2.54mm:PinHeader_1x06_P2.54mm_Vertical, symbol Connector_Generic:Conn_01x06
- added C1: 100nf, Capacitor_SMD:C_0805_2012Metric_Pad1.18x1.45mm_HandSolder, symbol Device:C
- added R1: 10K, Resistor_SMD:R_0805_2012Metric_Pad1.20x1.40mm_HandSolder, symbol Device:R
- added R2: 470, Resistor_SMD:R_0805_2012Metric_Pad1.20x1.40mm_HandSolder, symbol Device:R
- added U2: 74HC138, Package_SO:SOIC-16_3.9x9.9mm_P1.27mm, symbol 74xx:74HC138
Connections:
- net DEVICE_ENABLE: now also U2.2 (A1)
- net DEVICE_ENABLE2: now also R1.1, U2.1 (A0)
- net DEVICE_ENABLE_D: now also U2.14 (~{Y1})
- net GND: now also C1.2, U2.4 (~{E0}), U2.5 (~{E1}), U2.8 (GND)
- net VCC: now also C1.1, R1.2, U2.16 (VCC), U2.6 (E2)
- net WR_PROTECT: now also R2.2; no longer J1.20 (Pin_20)
- net GND4 renamed EN35
- net EN35: now also U2.3 (A2)
- new net WR_PROTECT_D: J1.20 (Pin_20), R2.1
- no-connect marks 0 -> 7
